File: PCB/PCB.kicad_pcb (KiCad board)
At the start: 2 copper layers, 11 x 11.5 mm, 19 parts, among them U1 STM32G031F6P6, U2 A7106, U3 HT7333-3.3V, Y1 16MHz

Commit message: feat: Update PCB
Parts:
- C2, C6, C7, L1, R1, U1: moved to F.Cu
- moved R1 17.5 mm to (154.1, 88.4), turned to 0 degrees
- moved L1 15.9 mm to (154.1, 86.4), turned to 0 degrees
- moved Y1 15.8 mm to (142.5, 83.9)
- moved C7 15.1 mm to (141.9, 87.4)
- moved GND1 14.1 mm to (141.4, 80.1), turned to 0 degrees
- moved VCC1 13.5 mm to (144.5, 77.0)
- moved CH3 12.5 mm to (141.4, 77.0), turned to 0 degrees
- moved CH1 12.5 mm to (141.4, 70.9), turned to 0 degrees
- moved CH2 12.0 mm to (141.4, 74.0), turned to 0 degrees
- moved U3 9.35 mm to (156.0, 82.3), turned to 0 degrees
- moved U2 8.99 mm to (149.5, 82.4)
- moved TP1 8.26 mm to (144.5, 70.9), turned to 0 degrees
- moved C3 7.90 mm to (147.5, 72.4), turned to 0 degrees
- moved TP2 7.84 mm to (144.5, 74.0), turned to 0 degrees
- moved C4 7.51 mm to (147.5, 74.3), turned to 0 degrees
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Routing:
- net Net-(U1-VSS): track 0.00 -> 42.2 mm, vias 0 -> 4
- net Net-(U2-DVDD): track 0.00 -> 34.2 mm, vias 0 -> 3
- net Net-(U3-VIN): track 0.00 -> 22.2 mm, vias 0 -> 2
- net Net-(U1-PA13): track 0.00 -> 21.1 mm, vias 0 -> 2
- net Net-(U2-XO): track 0.00 -> 19.6 mm, vias 0 -> 2
- net Net-(U1-NRST): track 0.00 -> 19.5 mm
- net Net-(U1-PA3): track 0.00 -> 17.2 mm, vias 0 -> 2
- net Net-(C2-Pad2): track 0.00 -> 17.0 mm
- net Net-(U1-PB0): track 0.00 -> 15.0 mm, vias 0 -> 2
- net Net-(U1-PA14): track 0.00 -> 14.6 mm, vias 0 -> 2
- net Net-(U1-PA5): track 0.00 -> 14.3 mm, vias 0 -> 2
- net Net-(C3-Pad1): track 0.00 -> 13.7 mm
- net Net-(C7-Pad1): track 0.00 -> 13.7 mm, vias 0 -> 1
- net Net-(U1-PA1): track 0.00 -> 13.3 mm, vias 0 -> 1
- net Net-(U1-PA0): track 0.00 -> 12.1 mm, vias 0 -> 1
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Other:
- board size 11 x 11.5 mm -> 19 x 20 mm
- board text removed: "FS2A"

Commit message: PCB changes
Connections:
- L1 pad 2: unconnected-(L1-Pad2) -> ANTENNA

Commit message: Update PCB
Parts:
- moved TP1 13.6 mm to (133.6, 79.0)
- moved TP2 13.6 mm to (133.6, 82.1)
- moved C7 13.6 mm to (131.0, 95.5)
- moved U2 13.6 mm to (138.6, 90.5)
- moved VCC1 13.6 mm to (133.6, 85.1)
- moved CH1 13.6 mm to (130.5, 79.0)
- moved CH2 13.6 mm to (130.5, 82.1)
- moved L1 13.6 mm to (143.2, 94.5)
- moved U1 13.6 mm to (142.7, 81.5)
- moved U3 13.6 mm to (145.1, 90.5)
- moved C2 13.6 mm to (136.5, 78.5)
- moved C3 13.6 mm to (136.5, 80.5)
- moved C4 13.6 mm to (136.5, 82.4)
- moved C5 13.6 mm to (136.5, 84.4)
- moved C6 13.6 mm to (136.5, 86.4)
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Connections:
- L1 pad 2: ANTENNA -> unconnected-(L1-Pad2)
Routing:
- net Net-(U2-XI): track 0.00 -> 30.1 mm, vias 0 -> 2
- net Net-(U1-PA5): track 14.3 -> 0.00 mm, vias 2 -> 0
- net Net-(U2-RFO): track 10.4 -> 19.4 mm
- net Net-(U1-VSS): track 42.2 -> 49.9 mm, vias 4 -> 3
- net Net-(U1-PB0): track 15.0 -> 21.2 mm, vias 2 -> 4
- net Net-(U1-NRST): track 19.5 -> 13.2 mm
- net Net-(U3-VIN): track 22.2 -> 16.0 mm
- net Net-(U1-PA13): track 21.1 -> 15.5 mm, vias 2 -> 0
- net Net-(U1-PA3): track 17.2 -> 12.6 mm, vias 2 -> 0
- net Net-(U2-DVDD): track 34.2 -> 38.7 mm, vias 3 -> 4
- net Net-(C2-Pad2): track 17.0 -> 20.4 mm
- net Net-(U2-XO): track 19.6 -> 21.6 mm
- net Net-(U1-PA14): track 14.6 -> 13.1 mm
- net Net-(U1-PA1): track 13.3 -> 12.0 mm, vias 1 -> 0
- net Net-(C3-Pad1): track 13.7 -> 14.7 mm, vias 0 -> 2
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Other:
- board size 19 x 20 mm -> 19 x 19 mm

Commit message: feat: Update PCB
Parts:
- added C1: 2.7pF, Capacitor_SMD:C_0402_1005Metric, F.Cu at (138.0, 86.0)
- moved C5 9.64 mm to (138.0, 93.9)
- moved C6 9.64 mm to (138.0, 95.9)
- moved C2 9.64 mm to (138.0, 88.0)
- moved C3 9.64 mm to (138.0, 90.0)
- moved C4 9.64 mm to (138.0, 91.9)
- moved U2 4.94 mm to (143.0, 88.2)
- moved U3 4.55 mm to (142.8, 94.4)
- moved L1 4.46 mm to (147.1, 92.3)
- moved C7 1.58 mm to (132.5, 95.0)
- moved CH1 1.58 mm to (132.0, 78.5)
- moved CH2 1.58 mm to (132.0, 81.6)
- moved CH3 1.58 mm to (132.0, 84.6)
- moved GND1 1.58 mm to (132.0, 87.7)
- moved TP1 1.58 mm to (135.1, 78.5)
- moved TP2 1.58 mm to (135.1, 81.6)
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Connections:
- C2 pad 2: Net-(C2-Pad2) -> Net-(U1-VSS)
- C3 pad 1: Net-(C3-Pad1) -> Net-(U2-XO)
- C3 pad 2: Net-(U2-XO) -> Net-(U1-VSS)
- C4 pad 1: Net-(U2-DVDD) -> Net-(U2-VDA1)
- L1 pad 2: unconnected-(L1-Pad2) -> Net-(C1-Pad1)
- R1 pad 2: Net-(U2-DVDD) -> Net-(U2-VDA1)
- U2 pad 10: Net-(U2-DVDD) -> Net-(U2-VDA1)
- U2 pad 13: Net-(U2-DVDD) -> unconnected-(U2-DVDD-Pad13)
- U2 pad 20: Net-(U2-DVDD) -> Net-(U2-VDA1)
- U2 pad 3: unconnected-(U2-RFI-Pad3) -> Net-(ANT1-PCB_Trace)
- U2 pad 5: Net-(U2-DVDD) -> Net-(U2-VDA1)
- U3 pad 3: Net-(U2-DVDD) -> Net-(U2-VDA1)
- Y1 pad 1: Net-(C2-Pad2) -> Net-(U1-VSS)
- Y1 pad 2: Net-(C3-Pad1) -> Net-(U2-XO)
Routing:
- net Net-(U2-DVDD): track 38.7 -> 0.00 mm, vias 4 -> 0
- net Net-(U2-VDA1): track 0.00 -> 32.8 mm, vias 0 -> 3
- net Net-(U2-XI): track 30.1 -> 0.00 mm, vias 2 -> 0
- net Net-(U2-REGI): track 4.62 -> 31.4 mm, vias 0 -> 2
- net Net-(C1-Pad1): track 0.00 -> 23.5 mm, vias 0 -> 2
- net Net-(C2-Pad2): track 20.4 -> 0.00 mm
- net Net-(C3-Pad1): track 14.7 -> 0.00 mm, vias 2 -> 0
- net Net-(U1-PB0): track 21.2 -> 7.23 mm, vias 4 -> 0
- net Net-(U1-PA5): track 0.00 -> 13.9 mm, vias 0 -> 2
- net Net-(U1-VDD): track 5.40 -> 17.4 mm, vias 0 -> 2
- net Net-(U1-NRST): track 13.2 -> 25.0 mm
- net Net-(U1-PA14): track 13.1 -> 24.4 mm, vias 2 -> 0
- net Net-(U1-VSS): track 49.9 -> 60.4 mm, vias 3 -> 1
- net Net-(U2-RFO): track 19.4 -> 8.90 mm, vias 0 -> 2
- net Net-(U1-PA3): track 12.6 -> 18.6 mm, vias 0 -> 2
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Other:
- board size 19 x 19 mm -> 19 x 21 mm

Commit message: feat: Update PCB
Parts:
- removed C5: 100nF, Capacitor_SMD:C_0402_1005Metric
- added ANT1: RFANT3216120A5T, Inductor_SMD:L_1206_3216Metric, F.Cu at (151.0, 102.3)
- moved U1 16.2 mm to (155.7, 88.5)
- moved U3 15.6 mm to (158.1, 97.5)
- moved C7 13.7 mm to (144.0, 102.5)
- moved CH1 13.7 mm to (143.5, 86.0)
- moved CH2 13.7 mm to (143.5, 89.1)
- moved CH3 13.7 mm to (143.5, 92.1)
- moved GND1 13.7 mm to (143.5, 95.2)
- moved TP1 13.7 mm to (146.6, 86.0)
- moved TP2 13.7 mm to (146.6, 89.1)
- moved VCC1 13.7 mm to (146.6, 92.1)
- moved Y1 13.7 mm to (144.6, 99.0)
- moved L1 12.9 mm to (156.2, 101.5)
- moved R1 12.9 mm to (156.2, 103.5)
- moved U2 12.7 mm to (151.6, 97.5)
- moved C6 11.8 mm to (149.5, 93.4)
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Connections:
- net Net-(U1-PA3) renamed /SCS
- net Net-(U1-PA5) renamed /SCK
- U2 pad 19: Net-(U2-REGI) -> unconnected-(U2-REGI-Pad19)
Routing:
- net Net-(U1-VSS): track 60.4 -> 0.00 mm, vias 1 -> 0
- net Net-(U2-VDA1): track 32.8 -> 0.00 mm, vias 3 -> 0
- net Net-(U2-REGI): track 31.4 -> 0.00 mm, vias 2 -> 0
- net Net-(U1-NRST): track 25.0 -> 0.00 mm
- net Net-(U1-PA14): track 24.4 -> 0.00 mm
- net Net-(C1-Pad1): track 23.5 -> 0.00 mm, vias 2 -> 0
- net /SCS: track 18.6 -> 0.00 mm, vias 2 -> 0
- net Net-(U1-VDD): track 17.4 -> 0.00 mm, vias 2 -> 0
- net Net-(U2-XO): track 16.3 -> 0.00 mm, vias 2 -> 0
- net /SCK: track 13.9 -> 0.00 mm, vias 2 -> 0
- net Net-(U1-PA13): track 12.2 -> 0.00 mm
- net Net-(U1-PA6): track 12.1 -> 0.00 mm, vias 2 -> 0
- net Net-(C7-Pad1): track 11.8 -> 0.00 mm
- net Net-(U1-PA7): track 11.6 -> 0.00 mm, vias 2 -> 0
- net Net-(U3-VIN): track 10.7 -> 0.00 mm
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Other:
- board outline removed

Commit message: Blank PCB state
Parts:
- moved CH3 23.4 mm to (166.0, 98.5), turned to 90 degrees
- moved CH2 21.6 mm to (163.0, 98.5), turned to 90 degrees
- moved CH1 20.7 mm to (160.0, 98.5), turned to 90 degrees
- moved GND1 13.9 mm to (157.0, 98.5)
- moved VCC1 9.79 mm to (154.0, 98.5)
- moved L1 8.48 mm to (147.7, 101.1)
- moved R1 8.48 mm to (147.7, 103.1)
- moved ANT1 8.48 mm to (142.5, 102.0)
- moved C1 8.48 mm to (141.1, 85.1)
- moved C2 8.48 mm to (141.1, 87.1)
- moved C3 8.48 mm to (141.1, 89.1)
- moved C4 8.48 mm to (141.1, 91.0)
- moved C6 8.48 mm to (141.1, 93.0)
- moved C7 8.48 mm to (135.5, 102.2)
- moved TP1 8.48 mm to (138.1, 85.7)
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Connections:
- net Net-(U1-PA6) renamed /SDIO
- net Net-(U1-PA7) renamed /GIO1
Other:
- board outline added: 14 x 15 mm
