File: PCB/PCB.kicad_pcb (KiCad board)
At the start: 2 copper layers, 14 x 15 mm, 20 parts, among them U1 STM32G031F6P6, U2 A7106, U3 HT7333-3.3V, Y1 16MHz

Commit message: Organise the schematic
Parts:
- removed CH1: Channel 1, TestPoint:TestPoint_THTPad_1.0x1.0mm_Drill0.5mm
- removed CH2: Channel 2, TestPoint:TestPoint_THTPad_1.0x1.0mm_Drill0.5mm
- removed CH3: Channel 3, TestPoint:TestPoint_THTPad_1.0x1.0mm_Drill0.5mm
- removed GND1: Ground, TestPoint:TestPoint_THTPad_1.0x1.0mm_Drill0.5mm
- removed VCC1: Power, TestPoint:TestPoint_THTPad_1.0x1.0mm_Drill0.5mm
- added C5: 100nF, Capacitor_SMD:C_0402_1005Metric, F.Cu at (199.5, 121.4)
- added J1: Conn_01x06_Pin, Connector_PinHeader_2.54mm:PinHeader_1x06_P2.54mm_Vertical, F.Cu at (195.8, 106.8)
- moved Y1 77.3 mm to (210.2, 120.9)
- moved TP1 73.5 mm to (208.7, 106.0)
- moved TP2 73.5 mm to (208.7, 109.1)
- moved C6 65.9 mm to (199.5, 123.4)
- moved C1 65.0 mm to (199.5, 113.5)
- moved C2 65.0 mm to (199.5, 115.5)
- moved C3 65.0 mm to (199.5, 117.5)
- moved C4 65.0 mm to (199.5, 119.4)
- moved L1 64.2 mm to (211.7, 105.5)
- moved R1 64.2 mm to (211.7, 107.5)
- moved ANT1 64.1 mm to (203.8, 120.5)
- moved U2 64.1 mm to (204.5, 115.7)
- moved U3 64.1 mm to (211.0, 115.7)
- moved C7 63.5 mm to (195.5, 123.0)
- moved U1 59.2 mm to (202.8, 108.5)
Connections:
- net Net-(U1-PB0) renamed /GIO2
- net Net-(U1-VSS) renamed GND
- U2 pad 13: unconnected-(U2-DVDD-Pad13) -> Net-(U2-DVDD)
Routing:
- net GND: track 0.00 -> 88.0 mm, vias 0 -> 1
- net Net-(U2-VDA1): track 0.00 -> 38.9 mm, vias 0 -> 5
- net Net-(U2-RFO): track 0.00 -> 33.6 mm, vias 0 -> 2
- net Net-(U3-VIN): track 0.00 -> 30.4 mm
- net Net-(U2-XO): track 0.00 -> 26.0 mm, vias 0 -> 4
- net Net-(C1-Pad1): track 0.00 -> 19.7 mm, vias 0 -> 2
- net Net-(U2-BPBG): track 0.00 -> 17.6 mm, vias 0 -> 2
- net Net-(U2-XI): track 0.00 -> 16.9 mm, vias 0 -> 2
- net Net-(U1-VDD): track 0.00 -> 15.6 mm, vias 0 -> 2
- net Net-(J1-Pin_2): track 0.00 -> 14.6 mm
- net /SCS: track 0.00 -> 14.2 mm, vias 0 -> 2
- net /SCK: track 0.00 -> 12.4 mm, vias 0 -> 2
- net /SDIO: track 0.00 -> 11.9 mm, vias 0 -> 2
- net Net-(J1-Pin_5): track 0.00 -> 11.5 mm
- net Net-(J1-Pin_4): track 0.00 -> 9.64 mm
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Other:
- board size 14 x 15 mm -> 33 x 25.5 mm

Commit message: More schematic updates
Connections:
- C2 pad 1: Net-(U2-XI) -> Net-(U2-VT)
- C3 pad 1: Net-(U2-XO) -> Net-(C3-Pad1)
- C4 pad 1: Net-(U2-VDA1) -> +3.3V
- C6 pad 2: Net-(U2-BPBG) -> unconnected-(C6-Pad2)
- J1 pad 3: Net-(J1-Pin_3) -> /CH1
- J1 pad 4: Net-(J1-Pin_4) -> /CH2
- J1 pad 5: Net-(J1-Pin_5) -> /CH3
- J1 pad 6: unconnected-(J1-Pin_6-Pad6) -> /CH4
- L1 pad 1: Net-(U2-RFO) -> Net-(U2-BPBG)
- R1 pad 2: Net-(U2-VDA1) -> +3.3V
- U1 pad 2: Net-(J1-Pin_3) -> unconnected-(U1-PA0-Pad2)
- U1 pad 3: Net-(J1-Pin_4) -> unconnected-(U1-PA1-Pad3)
- U1 pad 4: Net-(J1-Pin_5) -> unconnected-(U1-PA2-Pad4)
- U2 pad 1: unconnected-(U2-RSSI-Pad1) -> Net-(ANT1-PCB_Trace)
- U2 pad 10: Net-(U2-VDA1) -> unconnected-(U2-VDA3-Pad10)
- U2 pad 19: unconnected-(U2-REGI-Pad19) -> Net-(U2-REGI)
- U2 pad 20: Net-(U2-VDA1) -> +3.3V
- U2 pad 3: Net-(ANT1-PCB_Trace) -> unconnected-(U2-RFI-Pad3)
- U2 pad 4: Net-(U2-RFO) -> unconnected-(U2-RFO-Pad4)
- U2 pad 5: Net-(U2-VDA1) -> +3.3V
- U2 pad 6: unconnected-(U2-VT-Pad6) -> Net-(U2-VT)
- U2 pad 7: GND -> Net-(C3-Pad1)
- U2 pad 8: Net-(U2-XI) -> +3.3V
- U2 pad 9: Net-(U2-XO) -> unconnected-(U2-XO-Pad9)
- U3 pad 3: Net-(U2-VDA1) -> +3.3V
- Y1 pad 2: Net-(U2-XO) -> Net-(C3-Pad1)
Routing:
- net (no net): track 0.00 -> 110.8 mm, vias 0 -> 11
- net Net-(U2-VDA1): track 38.9 -> 0.00 mm, vias 5 -> 0
- net Net-(U2-RFO): track 33.6 -> 0.00 mm, vias 2 -> 0
- net Net-(U2-BPBG): track 17.6 -> 51.2 mm, vias 2 -> 4
- net Net-(U2-XO): track 26.0 -> 0.00 mm, vias 4 -> 0
- net Net-(U2-XI): track 16.9 -> 0.00 mm, vias 2 -> 0
- net Net-(J1-Pin_5): track 11.5 -> 0.00 mm
- net Net-(J1-Pin_4): track 9.64 -> 0.00 mm
- net Net-(J1-Pin_3): track 7.75 -> 0.00 mm
